Commit message: add new IMU calibration, add robot description

File: ros2_ws/src/mini_robot/urdf/mini_robot.urdf.xacro (robot description, xacro)
@@ -9,12 +9,21 @@
   <xacro:property name="base_width" value="0.16"/>
   <xacro:property name="base_height" value="0.06"/>
-  <xacro:property name="wheel_radius" value="0.04025"/>
+  <xacro:property name="wheel_radius" value="0.0235"/>
   <xacro:property name="wheel_width" value="0.026"/>
   <!-- Left-to-right wheel contact patch distance: TRACK_WIDTH_MM / 1000. -->
   <xacro:property name="track" value="0.20"/>
-  <!-- Driven axle sits slightly ahead of centre so the caster trails it. -->
-  <xacro:property name="axle_x" value="0.03"/>
-  <xacro:property name="caster_x" value="-0.06"/>
+  <!-- The drive axle IS the origin. The Arduino integrates odometry from the
+       mean of the two wheel distances - i.e. the drive-axle midpoint - and the
+       serial bridge publishes exactly that as odom -> base_footprint. Any
+       offset here would put the model's centre of rotation somewhere the
+       odometry is not, which mis-places the laser whenever the robot turns. -->
+  <xacro:property name="axle_x" value="0.0"/>
+  <!-- Passive trolley caster, on the centreline, 100 mm behind the drive axle. -->
+  <xacro:property name="caster_x" value="-0.10"/>
   <xacro:property name="caster_radius" value="0.015"/>
+  <!-- COIN-D6 sits directly above the caster, 100 mm above the ground. -->
+  <xacro:property name="laser_height" value="0.10"/>
+  <!-- Body box is nominal/visual only; offset back so it spans axle to caster. -->
+  <xacro:property name="body_x" value="-0.035"/>
   <material name="body"><color rgba="0.15 0.35 0.65 1"/></material>
   <material name="wheel"><color rgba="0.05 0.05 0.05 1"/></material>
@@ -27,7 +36,7 @@
   </joint>
   <link name="base_link">
-    <visual><origin xyz="0 0 ${base_height/2}"/><geometry><box size="${base_length} ${base_width} ${base_height}"/></geometry><material name="body"/></visual>
-    <collision><origin xyz="0 0 ${base_height/2}"/><geometry><box size="${base_length} ${base_width} ${base_height}"/></geometry></collision>
-    <inertial><origin xyz="0 0 ${base_height/2}"/><mass value="2.0"/><inertia ixx="0.008" ixy="0" ixz="0" iyy="0.008" iyz="0" izz="0.012"/></inertial>
+    <visual><origin xyz="${body_x} 0 ${base_height/2}"/><geometry><box size="${base_length} ${base_width} ${base_height}"/></geometry><material name="body"/></visual>
+    <collision><origin xyz="${body_x} 0 ${base_height/2}"/><geometry><box size="${base_length} ${base_width} ${base_height}"/></geometry></collision>
+    <inertial><origin xyz="${body_x} 0 ${base_height/2}"/><mass value="2.0"/><inertia ixx="0.008" ixy="0" ixz="0" iyy="0.008" iyz="0" izz="0.012"/></inertial>
   </link>
   <!-- Wheel joint names must match the /joint_states the serial bridge
@@ -62,5 +71,5 @@
     <visual><geometry><cylinder radius="0.035" length="0.035"/></geometry><material name="sensor"/></visual>
   </link>
-  <joint name="laser_joint" type="fixed"><parent link="base_link"/><child link="laser"/><origin xyz="0.04 0 0.10" rpy="0 0 0"/></joint>
+  <joint name="laser_joint" type="fixed"><parent link="base_link"/><child link="laser"/><origin xyz="${caster_x} 0 ${laser_height - wheel_radius}" rpy="0 0 0"/></joint>
   <!-- MPU9250/9255/6500. Frame of the /imu/data message. -->
   <link name="imu_link"/>

Commit message: flip the back to front

File: ros2_ws/src/mini_robot/urdf/mini_robot.urdf.xacro (robot description, xacro)
@@ -1,8 +1,13 @@
 <?xml version="1.0"?>
 <!-- Two-wheel differential drive base: one driven wheel per side on the
-     transverse axis, plus a passive caster behind them for the third contact
-     point. Dimensions are nominal; the ones that actually matter to the
-     software are 'track' (must match TRACK_WIDTH_MM in the sketch) and
-     'wheel_radius' (must match WHEEL_DIAMETER_MM / 2). -->
+     transverse axis, plus a passive caster for the third contact point.
+     The LiDAR points along the caster end, so THAT end is the robot's front
+     and +x runs towards it: the caster leads and the drive axle trails. The
+     Arduino uses the opposite convention (its "forward" is the axle end);
+     serial_bridge's reverse_base_direction parameter is what reconciles the
+     two, and must stay in step with the signs below.
+     Dimensions are nominal; the ones that actually matter to the software are
+     'track' (must match TRACK_WIDTH_MM in the sketch) and 'wheel_radius'
+     (must match WHEEL_DIAMETER_MM / 2). -->
 <robot xmlns:xacro="http://www.ros.org/wiki/xacro" name="mini_robot">
   <xacro:property name="base_length" value="0.18"/>
@@ -19,11 +24,12 @@
        odometry is not, which mis-places the laser whenever the robot turns. -->
   <xacro:property name="axle_x" value="0.0"/>
-  <!-- Passive trolley caster, on the centreline, 100 mm behind the drive axle. -->
-  <xacro:property name="caster_x" value="-0.10"/>
+  <!-- Passive trolley caster, on the centreline, 100 mm ahead of the drive
+       axle: it is the leading end, under the LiDAR. -->
+  <xacro:property name="caster_x" value="0.10"/>
   <xacro:property name="caster_radius" value="0.015"/>
   <!-- COIN-D6 sits directly above the caster, 100 mm above the ground. -->
   <xacro:property name="laser_height" value="0.10"/>
-  <!-- Body box is nominal/visual only; offset back so it spans axle to caster. -->
-  <xacro:property name="body_x" value="-0.035"/>
+  <!-- Body box is nominal/visual only; offset forward so it spans axle to caster. -->
+  <xacro:property name="body_x" value="0.035"/>
   <material name="body"><color rgba="0.15 0.35 0.65 1"/></material>
   <material name="wheel"><color rgba="0.05 0.05 0.05 1"/></material>
@@ -66,12 +72,17 @@
     <origin xyz="${caster_x} 0 ${caster_radius - wheel_radius}" rpy="0 0 0"/>
   </joint>
-  <!-- COIN-D6. If a wall straight ahead does not appear at angle zero in
-       /scan, correct the yaw in this joint's rpy rather than in the driver. -->
+  <!-- COIN-D6, above the caster. The unit is mounted with its own zero facing
+       the caster end, i.e. along base_link +x, so no yaw offset is needed here.
+       If a wall straight ahead does not appear at angle zero in /scan, correct
+       the yaw in this joint's rpy rather than in the driver. -->
   <link name="laser">
     <visual><geometry><cylinder radius="0.035" length="0.035"/></geometry><material name="sensor"/></visual>
   </link>
   <joint name="laser_joint" type="fixed"><parent link="base_link"/><child link="laser"/><origin xyz="${caster_x} 0 ${laser_height - wheel_radius}" rpy="0 0 0"/></joint>
-  <!-- MPU9250/9255/6500. Frame of the /imu/data message. -->
+  <!-- MPU9250/9255/6500. Frame of the /imu/data message. The chip is mounted
+       facing the axle end, which is now the rear, so imu_link is yawed 180 deg
+       from base_link. The bridge republishes the Arduino's IMU fields
+       unchanged; this joint is what tells TF which way they point. -->
   <link name="imu_link"/>
-  <joint name="imu_joint" type="fixed"><parent link="base_link"/><child link="imu_link"/><origin xyz="0 0 ${base_height}" rpy="0 0 0"/></joint>
+  <joint name="imu_joint" type="fixed"><parent link="base_link"/><child link="imu_link"/><origin xyz="0 0 ${base_height}" rpy="0 0 ${pi}"/></joint>
 </robot>
